File: FT232eval.sch (KiCad schematic (older format))
At the start: 7 parts, among them P1 USB_OTG, U1 FT232RL

Commit message: Add board layout and gerber files
Parts:
- added C3: 10u, Capacitors_SMD:c_elec_4x5.7, symbol CP
- added C4, C5: 100n, Capacitors_SMD:C_0603_HandSoldering, symbol C
- added D1: green, LEDs:LED_0603, symbol LED
- added P2: CONN_01X03, Pin_Headers:Pin_Header_Straight_1x03, symbol CONN_01X03
- added P3, P4: CONN_01X08, Pin_Headers:Pin_Header_Straight_1x08, symbol CONN_01X08
- added R3: 1k, Resistors_SMD:R_0603_HandSoldering, symbol R
- C1: value C -> 100n; footprint (none) -> Capacitors_SMD:C_0603_HandSoldering
- C2: footprint (none) -> Capacitors_SMD:c_elec_4x5.7
- L1, R1, R2: footprint (none) -> Resistors_SMD:R_0603_HandSoldering
- P1: footprint (none) -> Connect:USB_Mini-B
- U1: footprint SSOP-28 -> Housings_SSOP:SSOP-28_5.3x10.2mm_Pitch0.65mm
Connections:
- net +5V: now also C3.1, C4.1, P2.1 (P1), P4.7 (P7), R3.1
- net GND: now also P1.6 (shield), C3.2, C4.2, C5.2, D1.1 (K), P4.8 (P8)
- net TXD: now reaches U1.1 (TXD)
- net TXD: now also P3.1 (P1)
- net DCD: now reaches U1.10 (DCD)
- net DCD: now also P3.7 (P7)
- net CTS: now reaches U1.11 (CTS)
- net CTS: now also P3.4 (P4)
- net CBUS4: now reaches U1.12 (CBUS4)
- net CBUS4: now also P4.5 (P5)
- net CBUS2: now reaches U1.13 (CBUS2)
- net CBUS2: now also P4.3 (P3)
- net CBUS3: now reaches U1.14 (CBUS3)
- net CBUS3: now also P4.4 (P4)
- net +3V3: now reaches U1.17 (3V3OUT)
- net +3V3: now also C5.1, P2.3 (P3), P4.6 (P6)
- net at C1.1, C2.1, U1.19 (~RESET~)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: now also P2.2 (P2)
- net DTR: now reaches U1.2 (DTR)
- net DTR: now also P3.5 (P5)
- net CBUS1: now reaches U1.22 (CBUS1)
- net CBUS1: now also P4.2 (P2)
- net CBUS0: now reaches U1.23 (CBUS0)
- net CBUS0: now also P4.1 (P1)
- net RTS: now reaches U1.3 (RTS)
- net RTS: now also P3.3 (P3)
- net RXD: now reaches U1.5 (RXD)
- net RXD: now also P3.2 (P2)
- net RI: now reaches U1.6 (RI)
- net RI: now also P3.8 (P8)
- net DCR: now reaches U1.9 (DCR)
- net DCR: now also P3.6 (P6)
- new net: D1.2 (A), R3.2
Other:
- moved on the sheet: C1
